File: hardware/v2.1/gps-v2.1.kicad_pcb (KiCad board)
At the start: 2 copper layers, 40 x 35 mm, 35 parts, among them P101 CON-SENSOR, P103 Boot, P104 U.FL, U101 XMC1302-32, U102 FireFlyX1, U103 DRILL, U104 DRILL, U105 DRILL, U106 DRILL

Commit message: v2.1 ready for prototype
Parts:
- L101: footprint kicad-libraries:C0603E -> kicad-libraries:R0603E
- turned FB101 to 90 degrees
Connections:
- BT101 pad 1: +BATT -> VBat
- C106 pad 2: Net-(C106-Pad2) -> VBat
- FB101 pad 1: Net-(C101-Pad2) -> VCC
- FB101 pad 2: VCC -> Net-(C101-Pad2)
- P104 pad 1: Net-(P104-Pad1) -> Net-(L101-Pad2)
- U102 pad 2: Net-(P104-Pad1) -> Net-(L101-Pad2)
- U102 pad 8: Net-(C106-Pad2) -> VBat
Routing:
- net VBat: track 0.00 -> 19.5 mm
- net +BATT: track 16.6 -> 0.00 mm
- net Net-(C106-Pad2): track 2.85 -> 0.00 mm
