File: hardware/gps-v2.1.kicad_pcb (KiCad board)
At the start: 2 copper layers, 40 x 35 mm, 35 parts, among them P101 CON-SENSOR, P103 Boot, P104 U.FL, U101 XMC1302-32, U102 FireFlyX1, U103 DRILL, U104 DRILL, U105 DRILL, U106 DRILL

Commit message: fix weee logo
Parts:
- VAL: value WEEE_7mm_back -> WEEE_7mm; footprint kicad-libraries:WEEE_7mm_back -> kicad-libraries:WEEE_7mm
- turned VAL to 180 degrees

Commit message: add battery description
Other:
- board text added: "CR1025"
Changed lines of the file:
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@@
-(kicad_pcb (version 20171130) (host pcbnew 5.1.4-e60b266~84~ubuntu18.04.1)
+(kicad_pcb (version 20171130) (host pcbnew 5.1.5-52549c5~84~ubuntu18.04.1)
   (general
     (thickness 1.6)
-    (drawings 20)
+    (drawings 21)
     (tracks 357)
     (zones 0)
@@
   (page A4)
   (layers
-    (0 F.Cu signal)
-    (31 B.Cu signal)
+    (0 F.Cu signal hide)
+    (31 B.Cu signal hide)
     (32 B.Adhes user hide)
     (33 F.Adhes user hide)
@@
     (aux_axis_origin 166.4 85.9)
     (grid_origin 166.4 85.9)
-    (visible_elements FFFFFF7F)
+    (visible_elements FFFEFF7F)
     (pcbplotparams
       (layerselection 0x011f8_ffffffff)
@@
     )
   )
+  (gr_text CR1025 (at 171.3 111.8) (layer F.SilkS)
+    (effects (font (size 0.8 0.8) (thickness 0.15)))
+  )
   (gr_line (start 188 89.9) (end 184.8 89.9) (angle 90) (layer Edge.Cuts) (width 0.15))
